Commit message: scene/gripper: change left_arm gripper to RG2

File: mime/assets/prl_ur5/robot.urdf (robot description, URDF)
Before this commit: robot prl_ur5_robot, 77 links, 76 joints
Links:
- removed link left_gripper_finger_1_safety_shield
- removed link left_gripper_finger_2_safety_shield
- link left_gripper_body: mass 0.78 -> 0.65; geometry collision mesh filename=./meshes/rg2_v1/collision/body.stl; visual mesh filename=./meshes/rg2_v1/visual/body.stl
- link left_gripper_bracket: mass 0.001 -> 0.09; geometry collision mesh filename=./meshes/rg2_v1/collision/single_bracket.stl; visual mesh filename=./meshes/rg2_v1/visual/single_bracket.stl
- link left_gripper_finger_1_finger_tip: geometry collision mesh filename=./meshes/rg2_v1/collision/finger_tip_1.stl; collision mesh filename=./meshes/rg2_v1/collision/finger_tip_2.stl
- link left_gripper_finger_1_flex_finger: geometry collision mesh filename=./meshes/rg2_v1/collision/flex_finger.stl; visual mesh filename=./meshes/rg2_v1/visual/flex_finger.stl
- link left_gripper_finger_1_moment_arm: geometry collision mesh filename=./meshes/rg2_v1/collision/moment_arm.stl; visual mesh filename=./meshes/rg2_v1/visual/moment_arm.stl
- link left_gripper_finger_1_truss_arm: geometry collision mesh filename=./meshes/rg2_v1/collision/truss_arm.stl; visual mesh filename=./meshes/rg2_v1/visual/truss_arm.stl
- link left_gripper_finger_2_finger_tip: geometry collision mesh filename=./meshes/rg2_v1/collision/finger_tip_1.stl; collision mesh filename=./meshes/rg2_v1/collision/finger_tip_2.stl
- link left_gripper_finger_2_flex_finger: geometry collision mesh filename=./meshes/rg2_v1/collision/flex_finger.stl; visual mesh filename=./meshes/rg2_v1/visual/flex_finger.stl
- link left_gripper_finger_2_moment_arm: geometry collision mesh filename=./meshes/rg2_v1/collision/moment_arm.stl; visual mesh filename=./meshes/rg2_v1/visual/moment_arm.stl
- link left_gripper_finger_2_truss_arm: geometry collision mesh filename=./meshes/rg2_v1/collision/truss_arm.stl; visual mesh filename=./meshes/rg2_v1/visual/truss_arm.stl
Joints:
- removed joint left_gripper_finger_1_safety_shield_joint
- removed joint left_gripper_finger_2_safety_shield_joint
- joint left_camera_joint: origin xyz=0.0 0.02 0.15 rpy=-1.57 -1.57 0.0 -> xyz=0.0 0.01 0.13 rpy=-1.57 -1.57 0.0
- joint left_gripper_body_joint: origin xyz=0.0 0.0 0.051 rpy=0.0 0.0 0.0 -> xyz=0.0 0.0 0.05 rpy=0.0 0.0 0.0
- joint left_gripper_finger_1_finger_tip_joint: limit lower=0.0 upper=1.3 effort=10.0 velocity=2.4 -> lower=0.0 upper=1.3 effort=2.2 velocity=0.5; origin xyz=-0.05503 0.0 0.05807 rpy=0.0 0.49 0.0 -> xyz=-0.0256 0.0 0.04868 rpy=0.0 0.772 0.0
- joint left_gripper_finger_1_flex_finger_joint: origin xyz=0.0098 0.0 0.0218 rpy=0.0 0.0 0.0 -> xyz=0.03059 0.0 0.0172 rpy=0.0 0.0 0.0
- joint left_gripper_finger_1_truss_arm_joint: limit lower=0.0 upper=1.3 effort=10.0 velocity=2.4 -> lower=0.0 upper=1.3 effort=2.2 velocity=0.5; origin xyz=-0.0105 0.0 0.0891 rpy=0.0 -0.49 0.0 -> xyz=-0.0075 0.0 0.0715 rpy=0.0 -0.772 0.0
- joint left_gripper_finger_2_finger_tip_joint: limit lower=0.0 upper=1.3 effort=10.0 velocity=2.4 -> lower=0.0 upper=1.3 effort=2.2 velocity=0.5; origin xyz=-0.05503 0.0 0.05807 rpy=0.0 0.49 0.0 -> xyz=-0.0256 0.0 0.04868 rpy=0.0 0.772 0.0
- joint left_gripper_finger_2_flex_finger_joint: origin xyz=0.0098 0.0 0.0218 rpy=0.0 0.0 0.0 -> xyz=0.03059 0.0 0.0172 rpy=0.0 0.0 0.0
- joint left_gripper_finger_2_truss_arm_joint: limit lower=0.0 upper=1.3 effort=10.0 velocity=2.4 -> lower=0.0 upper=1.3 effort=2.2 velocity=0.5; origin xyz=-0.0105 0.0 0.0891 rpy=0.0 -0.49 0.0 -> xyz=-0.0075 0.0 0.0715 rpy=0.0 -0.772 0.0
- joint left_gripper_grasp_frame_joint: origin xyz=0.0 0.0 0.19 rpy=0.0 0.0 0.0 -> xyz=0.0 0.0 0.14 rpy=0.0 0.0 0.0
- joint left_gripper_joint: limit lower=0.0 upper=1.3 effort=10.0 velocity=2.4 -> lower=0.0 upper=1.3 effort=2.2 velocity=0.5; origin xyz=-0.0238 0.0 0.066 rpy=0.0 -0.49 0.0 -> xyz=-0.017 0.0 0.055 rpy=0.0 -0.772 0.0
- joint left_gripper_mirror_joint: limit lower=0.0 upper=1.3 effort=10.0 velocity=2.4 -> lower=0.0 upper=1.3 effort=2.2 velocity=0.5; origin xyz=-0.0238 0.0 0.066 rpy=0.0 -0.49 0.0 -> xyz=-0.017 0.0 0.055 rpy=0.0 -0.772 0.0

Commit message: assets/prl_ur5/robot: update right gripper

File: mime/assets/prl_ur5/robot.urdf (robot description, URDF)
Before this commit: robot prl_ur5_robot, 75 links, 74 joints
Links:
- added link right_gripper_finger_1_safety_shield, mass 0.001; collision box size=0.0 0.0 0.0; visual mesh filename=./meshes/rg6_v1/visual/safety_shield.stl
- added link right_gripper_finger_2_safety_shield, mass 0.001; collision box size=0.0 0.0 0.0; visual mesh filename=./meshes/rg6_v1/visual/safety_shield.stl
- link right_gripper_body: mass 0.65 -> 0.78; geometry collision mesh filename=./meshes/rg6_v1/collision/body.stl; visual mesh filename=./meshes/rg6_v1/visual/body.stl
- link right_gripper_bracket: mass 0.09 -> 0.001; geometry collision mesh filename=./meshes/rg6_v1/collision/single_bracket.stl; visual mesh filename=./meshes/rg6_v1/visual/single_bracket.stl
- link right_gripper_finger_1_finger_tip: geometry collision mesh filename=./meshes/rg6_v1/collision/finger_tip_1.stl; collision mesh filename=./meshes/rg6_v1/collision/finger_tip_2.stl
- link right_gripper_finger_1_flex_finger: geometry collision mesh filename=./meshes/rg6_v1/collision/flex_finger.stl; visual mesh filename=./meshes/rg6_v1/visual/flex_finger.stl
- link right_gripper_finger_1_moment_arm: geometry collision mesh filename=./meshes/rg6_v1/collision/moment_arm.stl; visual mesh filename=./meshes/rg6_v1/visual/moment_arm.stl
- link right_gripper_finger_1_truss_arm: geometry collision mesh filename=./meshes/rg6_v1/collision/truss_arm.stl; visual mesh filename=./meshes/rg6_v1/visual/truss_arm.stl
- link right_gripper_finger_2_finger_tip: geometry collision mesh filename=./meshes/rg6_v1/collision/finger_tip_1.stl; collision mesh filename=./meshes/rg6_v1/collision/finger_tip_2.stl
- link right_gripper_finger_2_flex_finger: geometry collision mesh filename=./meshes/rg6_v1/collision/flex_finger.stl; visual mesh filename=./meshes/rg6_v1/visual/flex_finger.stl
- link right_gripper_finger_2_moment_arm: geometry collision mesh filename=./meshes/rg6_v1/collision/moment_arm.stl; visual mesh filename=./meshes/rg6_v1/visual/moment_arm.stl
- link right_gripper_finger_2_truss_arm: geometry collision mesh filename=./meshes/rg6_v1/collision/truss_arm.stl; visual mesh filename=./meshes/rg6_v1/visual/truss_arm.stl
Joints:
- added joint right_gripper_finger_1_safety_shield_joint: type revolute, parent right_gripper_finger_1_finger_tip, child right_gripper_finger_1_safety_shield, origin xyz=-0.00665 0.0 -0.01155 rpy=0.0 -0.49 0.0, axis 0 1 0, limit lower=0.0 upper=1.3 effort=10.0 velocity=2.4, mimic joint=right_gripper_joint multiplier=1 offset=0
- added joint right_gripper_finger_2_safety_shield_joint: type revolute, parent right_gripper_finger_2_finger_tip, child right_gripper_finger_2_safety_shield, origin xyz=-0.00665 0.0 -0.01155 rpy=0.0 -0.49 0.0, axis 0 1 0, limit lower=0.0 upper=1.3 effort=10.0 velocity=2.4, mimic joint=right_gripper_joint multiplier=1 offset=0
- joint right_camera_color_optical_joint: origin xyz=0 0 0 rpy=-1.5540411677948966 0.001 -1.5607963267948966 -> xyz=0 0 0 rpy=-1.5707963267948966 0 -1.5707963267948966
- joint right_camera_joint: origin xyz=0.0 0.01 0.13 rpy=-1.57 -1.57 0.0 -> xyz=0.0 0.02 0.15 rpy=-1.57 -1.57 0.0
- joint right_gripper_body_joint: origin xyz=0.0 0.0 0.05 rpy=0.0 0.0 0.0 -> xyz=0.0 0.0 0.051 rpy=0.0 0.0 0.0
- joint right_gripper_finger_1_finger_tip_joint: limit lower=0.0 upper=1.3 effort=2.2 velocity=0.5 -> lower=0.0 upper=1.3 effort=10.0 velocity=2.4; origin xyz=-0.0256 0.0 0.04868 rpy=0.0 0.772 0.0 -> xyz=-0.05503 0.0 0.05807 rpy=0.0 0.49 0.0
- joint right_gripper_finger_1_flex_finger_joint: origin xyz=0.03059 0.0 0.0172 rpy=0.0 0.0 0.0 -> xyz=0.0098 0.0 0.0218 rpy=0.0 0.0 0.0
- joint right_gripper_finger_1_truss_arm_joint: limit lower=0.0 upper=1.3 effort=2.2 velocity=0.5 -> lower=0.0 upper=1.3 effort=10.0 velocity=2.4; origin xyz=-0.0075 0.0 0.0715 rpy=0.0 -0.772 0.0 -> xyz=-0.0105 0.0 0.0891 rpy=0.0 -0.49 0.0
- joint right_gripper_finger_2_finger_tip_joint: limit lower=0.0 upper=1.3 effort=2.2 velocity=0.5 -> lower=0.0 upper=1.3 effort=10.0 velocity=2.4; origin xyz=-0.0256 0.0 0.04868 rpy=0.0 0.772 0.0 -> xyz=-0.05503 0.0 0.05807 rpy=0.0 0.49 0.0
- joint right_gripper_finger_2_flex_finger_joint: origin xyz=0.03059 0.0 0.0172 rpy=0.0 0.0 0.0 -> xyz=0.0098 0.0 0.0218 rpy=0.0 0.0 0.0
- joint right_gripper_finger_2_truss_arm_joint: limit lower=0.0 upper=1.3 effort=2.2 velocity=0.5 -> lower=0.0 upper=1.3 effort=10.0 velocity=2.4; origin xyz=-0.0075 0.0 0.0715 rpy=0.0 -0.772 0.0 -> xyz=-0.0105 0.0 0.0891 rpy=0.0 -0.49 0.0
- joint right_gripper_grasp_frame_joint: origin xyz=0.0 0.0 0.14 rpy=0.0 0.0 0.0 -> xyz=0.0 0.0 0.19 rpy=0.0 0.0 0.0
- joint right_gripper_joint: limit lower=0.0 upper=1.3 effort=2.2 velocity=0.5 -> lower=0.0 upper=1.3 effort=10.0 velocity=2.4; origin xyz=-0.017 0.0 0.055 rpy=0.0 -0.772 0.0 -> xyz=-0.0238 0.0 0.066 rpy=0.0 -0.49 0.0
- joint right_gripper_mirror_joint: limit lower=0.0 upper=1.3 effort=2.2 velocity=0.5 -> lower=0.0 upper=1.3 effort=10.0 velocity=2.4; origin xyz=-0.017 0.0 0.055 rpy=0.0 -0.772 0.0 -> xyz=-0.0238 0.0 0.066 rpy=0.0 -0.49 0.0
